File: vcf_as3320_lpf_v1/vcf_as3320_lpf_v1.kicad_sch (KiCad schematic)
At the start: 55 parts, among them J1 Conn_02x05_Odd_Even, J4 IN1, J5 OUT_2, U2 TL072, U3 AS3320, U4 LM79L05_TO92

Commit message: Draft layout done no routing
Parts:
- U4: footprint Package_TO_SOT_THT:TO-92_Inline -> Package_TO_SOT_THT:TO-92_Inline_Wide
Changed lines of the file:
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@@
     (property "Reference" "U4" (id 0) (at 160.02 19.7825 0))
     (property "Value" "LM79L05_TO92" (id 1) (at 160.02 22.5576 0))
-    (property "Footprint" "Package_TO_SOT_THT:TO-92_Inline" (id 2) (at 160.02 20.574 0)
+    (property "Footprint" "Package_TO_SOT_THT:TO-92_Inline_Wide" (id 2) (at 160.02 20.574 0)
       (effects (font (size 1.27 1.27) italic) hide)
     )
@@
     )
     (path "/8af282d4-ad28-4e3e-ab45-7b030865f8ef/606534f2-a8d4-469a-95d0-3918b850058b"
-      (reference "D1") (unit 1) (value "D") (footprint "Diode_THT:D_A-405_P7.62mm_Horizontal")
+      (reference "D1") (unit 1) (value "D") (footprint "Diode_THT:D_A-405_P2.54mm_Vertical_KathodeUp")
     )
     (path "/06f573de-ffb2-4af5-8c31-cc321694122a"
@@
     )
     (path "/8af282d4-ad28-4e3e-ab45-7b030865f8ef/57426924-16dd-40e4-87cb-c1b513f62ba3"
-      (reference "D4") (unit 1) (value "D") (footprint "Diode_THT:D_A-405_P7.62mm_Horizontal")
+      (reference "D4") (unit 1) (value "D") (footprint "Diode_THT:D_A-405_P2.54mm_Vertical_KathodeUp")
     )
     (path "/3c5c2fda-68a3-437c-bc2c-ea7802ac1a5e"
@@
       (reference "J5") (unit 1) (value "OUT_2") (footprint "My Stuff:Jack_3.5mm_MJ-355W_Vertical")
     )
-    (path "/8af282d4-ad28-4e3e-ab45-7b030865f8ef/3ca7e2ef-f59b-48e7-8123-cdab6fbab32e"
-      (reference "J_FREQ1") (unit 1) (value "FREQ") (footprint "My Stuff:Jack_3.5mm_MJ-355W_and_PJ398SM_Vertical")
-    )
-    (path "/8af282d4-ad28-4e3e-ab45-7b030865f8ef/feccf875-5dd5-45fa-aad9-80e8723adba1"
-      (reference "J_FREQ2") (unit 1) (value "FREQ") (footprint "My Stuff:Jack_3.5mm_MJ-355W_and_PJ398SM_Vertical")
+    (path "/8af282d4-ad28-4e3e-ab45-7b030865f8ef/d5e790bc-2d50-4d2e-a686-b171b678254e"
+      (reference "J_FREQ1") (unit 1) (value "FREQ") (footprint "My Stuff:Jack_3.5mm_MJ-355W_Vertical")
+    )
+    (path "/8af282d4-ad28-4e3e-ab45-7b030865f8ef/36f54cc5-468c-4db1-97d8-92803f64a56d"
+      (reference "J_RES1") (unit 1) (value "RES") (footprint "My Stuff:Jack_3.5mm_MJ-355W_Vertical")
     )
     (path "/fb718fde-b64d-4cc3-b404-7e5f0c9c36ea"
@@
     )
     (path "/8de01783-4451-4607-a8ef-114f3601b521"
-      (reference "U4") (unit 1) (value "LM79L05_TO92") (footprint "Package_TO_SOT_THT:TO-92_Inline")
+      (reference "U4") (unit 1) (value "LM79L05_TO92") (footprint "Package_TO_SOT_THT:TO-92_Inline_Wide")
     )
     (path "/8af282d4-ad28-4e3e-ab45-7b030865f8ef/916f16bd-1c8e-4c0c-bdbb-3c7f6e4f6f3d"

Commit message: Geographic rename, silkscreen cleanup
Parts:
- D2, D3: value D -> 1N4001
- renumbered C14 to C10, C9 to C11, C10 to C12, C12 to C13, C11 to C14, C17 to C15, C19 to C17, C3 to C18, C8 to C19, C15 to C20, C7 to C21, C4 to C3, C5 to C4, C1 to C5, C2 to C6, C13 to C9, R23 to R21, R21 to R23, R14 to R24, R20 to R25, R19 to R26, R17 to R27, R18 to R28, R11 to R29, R16 to R30, RB3 to RB1, RB1 to RB3, RC3 to RC2, RC2 to RC3, RC1 to RC4, RF4 to RF1, RF3 to RF2, RF2 to RF3, RF1 to RF4
Other:
- title: (none) -> VCF AS3320
